Commit message: update diffbot.urdf.xacro

File: urdf/diffbot.urdf.xacro (robot description, xacro)
@@ -1,8 +1,9 @@
 <?xml version="1.0"?>
 <robot xmlns:xacro="http://www.ros.org/wiki/xacro" name="mobile_robot">
-  <xacro:property name="package_name" value="mobile_robot_description"/>
+  <xacro:property name="package_name" value="diffbot_description"/>
   <xacro:property name="robot_name" value="diffbot"/>
   <xacro:include filename="$(find ${package_name})/urdf/include/common_macros.urdf.xacro" />
-  <!-- <xacro:set_package_name /> -->
+  <xacro:include filename="$(find ${package_name})/urdf/include/common_sensors.xacro" />
+  <xacro:include filename="$(find ${package_name})/urdf/quimera_robot.gazebo.xacro" />
   <xacro:property name="caster_wheel_yaml" value="$(find ${package_name})/config/${robot_name}/caster_wheel.yaml" />
   <xacro:property name="caster_wheel_props" value="${load_yaml(caster_wheel_yaml)}"/>

Commit message: merge master to include motors

File: urdf/diffbot.urdf.xacro (robot description, xacro)
@@ -1,13 +1,15 @@
 <?xml version="1.0"?>
-<robot xmlns:xacro="http://www.ros.org/wiki/xacro" name="mobile_robot">
+<robot xmlns:xacro="http://www.ros.org/wiki/xacro" name="diffbot">
   <xacro:property name="package_name" value="diffbot_description"/>
   <xacro:property name="robot_name" value="diffbot"/>
   <xacro:include filename="$(find ${package_name})/urdf/include/common_macros.urdf.xacro" />
   <xacro:include filename="$(find ${package_name})/urdf/include/common_sensors.xacro" />
-  <xacro:include filename="$(find ${package_name})/urdf/quimera_robot.gazebo.xacro" />
+  <xacro:include filename="$(find ${package_name})/urdf/diffbot.gazebo.xacro" />
   <xacro:property name="caster_wheel_yaml" value="$(find ${package_name})/config/${robot_name}/caster_wheel.yaml" />
   <xacro:property name="caster_wheel_props" value="${load_yaml(caster_wheel_yaml)}"/>
   <xacro:property name="front_wheel_yaml" value="$(find ${package_name})/config/${robot_name}/front_wheel.yaml" />
   <xacro:property name="front_wheel_props" value="${load_yaml(front_wheel_yaml)}"/>
+  <xacro:property name="motor_yaml" value="$(find ${package_name})/config/${robot_name}/motor.yaml" />
+  <xacro:property name="motor_props" value="${load_yaml(motor_yaml)}"/>
   <xacro:property name="base_yaml" value="$(find ${package_name})/config/${robot_name}/base.yaml" />
   <xacro:property name="base_props" value="${load_yaml(base_yaml)}"/>
@@ -31,4 +33,15 @@
                       mesh="${front_wheel_props['wheel']['mesh']}">
   </xacro:wheel>
+  <!-- Motors -->
+  <xacro:motor prefix="right" reflect="-1"
+                      motor_props="${motor_props}"
+                      base_props="${base_props}"
+                      mesh="${motor_props['mesh']}">
+  </xacro:motor>
+  <xacro:motor prefix="left" reflect="1"
+                      motor_props="${motor_props}"
+                      base_props="${base_props}"
+                      mesh="${motor_props['mesh']}">
+  </xacro:motor>
   <!-- <xacro:include filename="$(find mobile_description)/urdf/mobile_robot_gazebo_plugins.xacro"/>  -->
 </robot>

Commit message: add base footprint link/joint

File: urdf/diffbot.urdf.xacro (robot description, xacro)
@@ -14,4 +14,6 @@
   <xacro:property name="base_yaml" value="$(find ${package_name})/config/${robot_name}/base.yaml" />
   <xacro:property name="base_props" value="${load_yaml(base_yaml)}"/>
+  <!-- Footprint link -->
+  <xacro:footprint wheel_props="${front_wheel_props}" />
   <!-- Base link -->
   <xacro:base base_prop="${base_props}" mesh="${base_props['base']['mesh']}" >
@@ -44,4 +46,4 @@
                       mesh="${motor_props['mesh']}">
   </xacro:motor>
-  <!-- <xacro:include filename="$(find mobile_description)/urdf/mobile_robot_gazebo_plugins.xacro"/>  -->
+  <!-- Sensors -->
 </robot>

File: urdf/include/common_macros.urdf.xacro (robot description, xacro)
@@ -314,4 +314,34 @@
     </link>
   </xacro:macro>
+<!-- ===================== Footprint xacro ==========================================
+  Xacro to create the base link. For more detail information and usage, see:
+    https://github.com/pxalcantara/mobile_robot_description/wiki/Base-xacro
+  params:
+  - base_props [dictionary]: base link properties;
+  - mesh [string]: file name of the link mesh;
+    - DEFAULT Value -> Empty string
+  - origin [block]: origin, position and orientation of the link;
+-->
+  <xacro:macro name="footprint"
+               params="wheel_props">
+    <!-- Base-Footprint -->
+    <!-- base_footprint is a fictitious link(frame) that is on the ground right below base_link origin -->
+    <link name="base_footprint">
+      <collision>
+        <!-- origin xyz="0 0 ${-base_z_origin_to_wheel_origin}" rpy="0 0 0" /-->
+        <origin xyz="0 0 ${wheel_props['wheel']['z_offset']}" rpy="0 0 0" />
+        <geometry>
+          <box size="0.001 0.001 0.001" />
+        </geometry>
+      </collision>
+    </link>
+    <!-- Joint to connect base_footprint with base_link -->
+    <joint name="base_footprint_joint" type="fixed">
+      <!-- origin xyz="0 0 ${wheel_radius - base_z_origin_to_wheel_origin}" rpy="0 0 0" /-->
+      <origin xyz="0 0 ${wheel_props['wheel']['radius'] - wheel_props['wheel']['z_offset']}" rpy="0 0 0" />
+      <parent link="base_footprint"/>
+      <child link="base_link" />
+    </joint>
+  </xacro:macro>
 <!-- ======================================================================= -->
 <!-- ======================= Intertial macros ===============================-->
